Commit message: state machine

File: environment/urdf/objects/slab3.urdf (robot description, URDF)
Before this commit: robot slab3, 1 links, 0 joints
Links:
- link slab3: geometry collision box size=0.005 0.29 0.2; visual box size=0.005 0.29 0.2

File: environment/urdf/objects/slab4.urdf (robot description, URDF)
Before this commit: robot slab4, 1 links, 0 joints
Links:
- link slab4: geometry collision box size=0.005 0.35 0.2; visual box size=0.005 0.35 0.2
